File: 0001-555-latches/0001-555-latches.kicad_sch (KiCad schematic)
At the start: 33 parts, among them J1 DC_IN, J2 ASTBL_OUT, J3 BSTBL_OUT, J4 MSTBL_OUT, SW1 SW_Push, SW2 SW_Push, SW3 SW_Push, U1 NE555P, U2 NE555P, U3 NE555P

Commit message: PCB labels (copper/silk)
Other:
- company: https://github.com/marcinciapa-el/0001 -> ${GH_REPO}
Changed lines of the file:
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@@
 	(title_block
 		(title "555 Latches")
-		(date "2025-10-08")
-		(rev "v0.0.1")
-		(company "https://github.com/marcinciapa-el/0001")
+		(date "${CURRENT_DATE}")
+		(rev "${VERSION}")
+		(company "${GH_REPO}")
 	)
 	(junction
