File: 0001-555-latches/0001-555-latches.kicad_pcb (KiCad board)
At the start: 2 copper layers, 37 parts, among them J1 DC_IN, J2 ASTBL_OUT, J3 BSTBL_OUT, J4 MSTBL_OUT, SW1 SW_Push, SW2 SW_Push, SW3 SW_Push, U1 NE555P, U2 NE555P, U3 NE555P

Commit message: PCB labels (copper/silk)
Parts:
- moved REF** 0.30 mm to (183.6, 129.2)
- moved REF** 0.30 mm to (106.4, 129.2)
Routing:
- net GND: track 584.1 -> 595.0 mm
- net Net-(U3-TR): track 50.3 -> 49.0 mm
Other:
- board text added: "${GH_REPO} REV:${VERSION} MK:XX"
- board text added: "ASTBL_OUT"
- board text added: "BSTBL_OUT"
- board text added: "MSTBL_OUT"
Changed lines of the file:
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@@
 	)
 	(paper "A4")
+	(title_block
+		(title "${PROJECTNAME}")
+		(date "${CURRENT_DATE}")
+		(rev "${VERSION}")
+		(company "${GH_REPO}")
+	)
 	(layers
 		(0 "F.Cu" signal)
@@
 		)
 	)
+	(property "GH_REPO" "https://github.com/marcinciapa-el/0001")
+	(property "VERSION" "1.0.0")
 	(net 0 "")
 	(net 1 "GND")
@@
 	(footprint "MountingHole:MountingHole_3.2mm_M3_Pad"
 		(layer "F.Cu")
-		(at 106.4 128.9)
+		(at 106.4 129.199058)
 		(descr "Mounting Hole 3.2mm, M3, generated by kicad-footprint-generator mountinghole.py")
 		(tags "mountinghole M3")
@@
 	(footprint "MountingHole:MountingHole_3.2mm_M3_Pad"
 		(layer "F.Cu")
-		(at 183.6 128.9)
+		(at 183.587569 129.199058)
 		(descr "Mounting Hole 3.2mm, M3, generated by kicad-footprint-generator mountinghole.py")
 		(tags "mountinghole M3")
@@
 		(embedded_fonts no)
 	)
-	(segment
-		(start 185.248218 61)
-		(end 188.345683 64.097465)
-		(width 2)
+	(gr_text "${GH_REPO}\nREV:${VERSION}\nMK:XX"
+		(at 178.956088 132.975496 0)
 		(layer "B.Cu")
-		(net 1)
+		(effects
+			(font
+				(size 1.3 1.3)
+				(thickness 0.1875)
+			)
+			(justify left bottom mirror)
+		)
+	)
+	(gr_text "MSTBL_OUT"
+		(at 188 125 90)
+		(layer "F.SilkS")
+		(effects
+			(font
+				(size 1 1)
+				(thickness 0.1)
+			)
+			(justify left bottom)
+		)
+	)
+	(gr_text "BSTBL_OUT"
+		(at 188 107 90)
+		(layer "F.SilkS")
+		(effects
+			(font
+				(size 1 1)
+				(thickness 0.1)
+			)
+			(justify left bottom)
+		)
+	)
+	(gr_text "ASTBL_OUT"
+		(at 188 88 90)
+		(layer "F.SilkS")
+		(effects
+			(font
+				(size 1 1)
+				(thickness 0.1)
+			)
+			(justify left bottom)
+		)
+	)
+	(gr_text "${GH_REPO}\nREV:${VERSION}\nMK:XX"
+		(at 111 133 0)
+		(layer "F.SilkS")
+		(effects
+			(font
+				(size 1 1)
+				(thickness 0.1)
+			)
+			(justify left bottom)
+		)
 	)
 	(segment
@@
 	)
 	(segment
+		(start 131 129)
+		(end 131 133.973046)
+		(width 1)
+		(layer "B.Cu")
+		(net 1)
+	)
+	(segment
 		(start 115.845683 109.808634)
 		(end 138 109.808634)
@@
 	)
 	(segment
-		(start 104.452782 133.601)
-		(end 185.547218 133.601)
-		(width 2)
+		(start 171.580571 106.543522)
+		(end 171.345683 106.308634)
+		(width 1)
 		(layer "B.Cu")
 		(net 1)
 	)
 	(segment
-		(start 171.580571 106.543522)
-		(end 171.345683 106.308634)
-		(width 1)
+		(start 188.301 130.699)
+		(end 188.345683 130.654317)
+		(width 2)
 		(layer "B.Cu")
 		(net 1)
@@
 	)
 	(segment
-		(start 145 61)
-		(end 150 61)
+		(start 188.345683 64.097465)
+		(end 185.447029 61.198811)
 		(width 2)
 		(layer "B.Cu")
@@
 	)
 	(segment
-		(start 188.345683 130.654317)
-		(end 188.345683 119.308634)
-		(width 2)
-		(layer "B.Cu")
-		(net 1)
-	)
-	(segment
-		(start 188.301 130.847218)
-		(end 188.301 130.699)
+		(start 188.345683 77.308634)
+		(end 188.345683 64.097465)
 		(width 2)
 		(layer "B.Cu")
@@
 	)
 	(segment
-		(start 140 61)
-		(end 140 70.7)
-		(width 2)
-		(layer "B.Cu")
-		(net 1)
-	)
-	(segment
 		(start 188.345683 117.308634)
 		(end 188.345683 116)
@@
 	)
 	(segment
-		(start 148 123.278517)
-		(end 148 134)
-		(width 1)
-		(layer "B.Cu")
-		(net 1)
-	)
-	(segment
 		(start 188.345683 108.308634)
 		(end 188.037049 108)
@@
 	)
 	(segment
-		(start 188.301 130.699)
-		(end 188.345683 130.654317)
+		(start 141 61.198811)
+		(end 104.552971 61.198811)
+		(width 2)
+		(layer "B.Cu")
+		(net 1)
+	)
+	(segment
+		(start 104.552971 61.198811)
+		(end 101.345683 64.406099)
 		(width 2)
 		(layer "B.Cu")
@@
 	)
 	(segment
-		(start 166 107)
-		(end 162 107)
+		(start 188.301 131.133845)
+		(end 188.301 130.699)
 		(width 2)
 		(layer "B.Cu")
@@
 	)
 	(segment
-		(start 101.345683 76.9)
-		(end 101.345683 64.406099)
+		(start 166 107)
+		(end 162 107)
 		(width 2)
 		(layer "B.Cu")
@@
 	)
 	(segment
-		(start 188.345683 64.097465)
-		(end 188.345683 77.308634)
-		(width 2)
-		(layer "B.Cu")
-		(net 1)
-	)
-	(segment
 		(start 114.345683 108.308634)
 		(end 115.845683 109.808634)
@@
 	)
 	(segment
+		(start 101.345683 121)
+		(end 101.345683 130.845683)
+		(width 2)
+		(layer "B.Cu")
+		(net 1)
+	)
+	(segment
 		(start 188.253722 80.400595)
 		(end 188.345683 80.308634)
@@
 	)
 	(segment
+		(start 136.721483 123.278517)
+		(end 131 129)
+		(width 1)
+		(layer "B.Cu")
+		(net 1)
+	)
+	(segment
 		(start 187.8758 120.778517)
 		(end 188.345683 120.308634)
@@
 	)
 	(segment
-		(start 145 61)
-		(end 145 68)
+		(start 101.345683 130.845683)
+		(end 104.473046 133.973046)
 		(width 2)
 		(layer "B.Cu")
@@
 	)
 	(segment
-		(start 101.345683 130.493901)
-		(end 104.452782 133.601)
-		(width 2)
-		(layer "B.Cu")
-		(net 1)
-	)
-	(segment
 		(start 180.845683 78.308634)
 		(end 187.345683 78.308634)
@@
 	)
 	(segment
-		(start 101.345683 121)
-		(end 101.345683 130.493901)
-		(width 2)
-		(layer "B.Cu")
-		(net 1)
-	)
-	(segment
 		(start 188.315566 119.278517)
 		(end 188.345683 119.308634)
@@
 	)
 	(segment
+		(start 101.345683 64.406099)
+		(end 101.345683 76.9)
+		(width 2)
+		(layer "B.Cu")
+		(net 1)
+	)
+	(segment
 		(start 179.735415 75.606687)
 		(end 179.735415 77.198366)
@@
 	)
 	(segment
-		(start 101.345683 64.406099)
-		(end 104.751782 61)
+		(start 131 133.973046)
+		(end 185.461799 133.973046)
+		(width 2)
+		(layer "B.Cu")
+		(net 1)
+	)
+	(segment
+		(start 188.345683 130.654317)
+		(end 188.345683 119.308634)
 		(width 2)
 		(layer "B.Cu")
@@
 	)
 	(segment
+		(start 144.646456 123.278517)
+		(end 136.721483 123.278517)
+		(width 1)
+		(layer "B.Cu")
+		(net 1)
+	)
+	(segment
+		(start 140.3 61.898811)
+		(end 141 61.198811)
+		(width 2)
+		(layer "B.Cu")
+		(net 1)
+	)
+	(segment
 		(start 179.685683 94.308634)
 		(end 179.685683 96.208634)
@@
 	)
 	(segment
-		(start 150 61)
-		(end 185.248218 61)
+		(start 145 61.198811)
+		(end 141 61.198811)
 		(width 2)
 		(layer "B.Cu")
@@
 	)
 	(segment
+		(start 104.473046 133.973046)
+		(end 131 133.973046)
+		(width 2)
+		(layer "B.Cu")
+		(net 1)
+	)
+	(segment
 		(start 142.845683 106.308634)
 		(end 144.646456 106.308634)
@@
 	)
 	(segment
-		(start 140 61)
-		(end 145 61)
-		(width 2)
-		(layer "B.Cu")
-		(net 1)
-	)
-	(segment
 		(start 182.57862 81.900595)
 		(end 184.07862 80.400595)
@@
 	)
 	(segment
-		(start 104.751782 61)
-		(end 140 61)
+		(start 140.3 71)
+		(end 140.3 61.898811)
+		(width 2)
+		(layer "B.Cu")
+		(net 1)
+	)
+	(segment
+		(start 145 61.198811)
+		(end 145 68)
+		(width 2)
+		(layer "B.Cu")
+		(net 1)
+	)
+	(segment
+		(start 185.447029 61.198811)
+		(end 145 61.198811)
 		(width 2)
 		(layer "B.Cu")
@@
 	)
 	(segment
-		(start 185.547218 133.601)
-		(end 188.301 130.847218)
+		(start 185.461799 133.973046)
+		(end 188.301 131.133845)
 		(width 2)
 		(layer "B.Cu")
@@
 	)
 	(segment
-		(start 127.845683 119.618634)
-		(end 127.845683 123.808634)
-		(width 0.6)
-		(layer "B.Cu")
-		(net 15)
-	)
-	(segment
-		(start 127.845683 127.808634)
-		(end 125.845683 129.808634)
-		(width 0.6)
-		(layer "B.Cu")
-		(net 15)
-	)
-	(segment
-		(start 127.845683 123.808634)
-		(end 127.845683 127.808634)
+		(start 143.424973 120)
+		(end 135 120)
 		(width 0.6)
 		(layer "B.Cu")
@@
 	)
 	(segment
-		(start 143.424973 120)
-		(end 135 120)
+		(start 135 120)
+		(end 130 125)
 		(width 0.6)
 		(layer "B.Cu")
@@
 	)
 	(segment
-		(start 135 120)
-		(end 133 122)
+		(start 125.191366 129.808634)
+		(end 118.845683 129.808634)
 		(width 0.6)
 		(layer "B.Cu")
@@
 	)
 	(segment
-		(start 118.845683 129.808634)
-		(end 116.885683 127.848634)
+		(start 130 125)
+		(end 125.191366 129.808634)
 		(width 0.6)
 		(layer "B.Cu")
@@
 	)
 	(segment
-		(start 127.845683 122)
-		(end 127.845683 123.808634)
+		(start 144.646456 118.778517)
+		(end 143.424973 120)
 		(width 0.6)
 		(layer "B.Cu")
@@
 	)
 	(segment
-		(start 125.845683 129.808634)
-		(end 118.845683 129.808634)
+		(start 127.845683 122.845683)
+		(end 130 125)
 		(width 0.6)
 		(layer "B.Cu")
@@
 	)
 	(segment
-		(start 133 122)
-		(end 127.845683 122)
+		(start 118.845683 129.808634)
+		(end 116.885683 127.848634)
 		(width 0.6)
 		(layer "B.Cu")
@@
 	)
 	(segment
-		(start 144.646456 118.778517)
-		(end 143.424973 120)
+		(start 127.845683 119.618634)
+		(end 127.845683 122.845683)
 		(width 0.6)
 		(layer "B.Cu")

Commit message: Closing PCB
Parts:
- removed REF** (x4): MountingHole_3.2mm_M3_Pad, MountingHole:MountingHole_3.2mm_M3_Pad
- added MNT1: MountingHole_3.2mm_M3_Pad, MountingHole:MountingHole_3.2mm_M3_Pad, F.Cu at (108.0, 68.0)
- added MNT2: MountingHole_3.2mm_M3_Pad, MountingHole:MountingHole_3.2mm_M3_Pad, F.Cu at (181.9, 68.0)
- added MNT3: MountingHole_3.2mm_M3_Pad, MountingHole:MountingHole_3.2mm_M3_Pad, F.Cu at (181.9, 129.0)
- added MNT4: MountingHole_3.2mm_M3_Pad, MountingHole:MountingHole_3.2mm_M3_Pad, F.Cu at (108.0, 129.0)
- moved J1 4.08 mm to (149.0, 75.0)
- moved R2 3.85 mm to (136.0, 79.3)
- moved J2 0.58 mm to (182.0, 85.4)
- moved J3 0.45 mm to (182.0, 104.1)
- moved J4 0.45 mm to (182.0, 122.8)
Routing:
- net GND: track 595.0 -> 576.6 mm
- net VCC: track 251.8 -> 256.3 mm
- net Net-(U1-THR): track 43.2 -> 39.8 mm
- net Net-(R2-Pad1): track 11.9 -> 14.8 mm
- net Net-(U1-DIS): track 51.4 -> 50.5 mm
- net /ASTBL_OUT: track 9.17 -> 8.59 mm
Other:
- board outline added: 88 x 75 mm
